File: kicad_project/MCU.kicad_sch (KiCad schematic)
At the start: 28 parts, among them IC1 ESP32-S3R8, SW1 B3U-1000P, SW2 B3U-1000P, Y1 40MHz

Commit message: Pcb to production
Parts:
- added R7: 10k, Resistor_SMD:R_0402_1005Metric, symbol Device:R
- added SW3: B3U-1000P, smd-non-ipc:B3U-1000P, symbol Switch:SW_Push
- C16, C17: LCSC Part # C161415 -> C161415
- DS1, R7: now not fitted; now left out of the parts list
- SW1, SW2: footprint hwlab:B3U-1000P -> smd-non-ipc:B3U-1000P
Connections:
- net +3V3: now also R7.1
- net GND: now also SW3.1
- net GPIO33: now reaches IC1.38 (GPIO33)
- net GPIO33: now also R7.2, SW3.2
- no-connect marks 5 -> 4
Other:
- note added: "MCU"
- note added: "ON/OFF DISPLAY"
